Commit message: Edit files to work in Gazebo Simulation

File: franka_description/robots/panda.transmission.xacro (robot description, xacro)
@@ -3,10 +3,10 @@
     <xacro:macro name="panda_transmission" params="robot_name">
         <!-- Load Gazebo lib and set the robot namespace -->
-        <gazebo>
+<!--         <gazebo>
             <plugin name="gazebo_ros_control" filename="libgazebo_ros_control.so">
-                <!-- <robotNamespace>/${robot_name}</robotNamespace> -->
+                <robotNamespace>/${robot_name}</robotNamespace>
  		             <legacyModeNS>false</legacyModeNS>
             </plugin>
-        </gazebo>
+        </gazebo> -->
         <transmission name="${robot_name}_tran_1">
             <type>transmission_interface/SimpleTransmission</type>

File: franka_description/robots/panda_arm.xacro (robot description, xacro)
@@ -29,242 +29,244 @@
   <xacro:property name="mass_link7" value="0.45606" />
   <xacro:property name="mass_link8" value="0.001" /> -->
-    <xacro:macro name="cylinder_inertial" params="radius length mass *origin">
-      <inertial>
-        <mass value="${mass}" />
-        <xacro:insert_block name="origin" />
-        <inertia ixx="${0.0833333 * mass * (3 * radius * radius + length * length)}" ixy="0.0" ixz="0.0"
-          iyy="${0.0833333 * mass * (3 * radius * radius + length * length)}" iyz="0.0"
-          izz="${0.5 * mass * radius * radius}" />
+  <xacro:macro name="cylinder_inertial" params="radius length mass *origin">
+    <inertial>
+      <mass value="${mass}" />
+      <xacro:insert_block name="origin" />
+      <inertia ixx="${0.0833333 * mass * (3 * radius * radius + length * length)}" ixy="0.0" ixz="0.0"
+        iyy="${0.0833333 * mass * (3 * radius * radius + length * length)}" iyz="0.0"
+        izz="${0.5 * mass * radius * radius}" />
       </inertial>
-  </xacro:macro>
-  <xacro:macro name="panda_arm" params="arm_id:='panda' description_pkg:='franka_description' connected_to:='' xyz:='0 0 0' rpy:='0 0 0'">
-    <xacro:unless value="${not connected_to}">
-      <joint name="${arm_id}_joint_${connected_to}" type="fixed">
-        <parent link="${connected_to}"/>
-        <child link="${arm_id}_link0"/>
-        <origin rpy="${rpy}" xyz="${xyz}"/>
-      </joint>
-    </xacro:unless>
-    <xacro:property name="joint_damping" value="1.0"/>
-    <joint name="robot_to_world" type="fixed">
-      <parent link="world" />
-      <child link="${arm_id}_link0" />
-      <origin xyz="0.0 0.0 0.0" rpy="0.0 0.0 0.0" />
-      <dynamics damping="${joint_damping}"/>
-    </joint>
-    <link name="${arm_id}_link0">
-      <visual>
-        <geometry>
-          <mesh filename="package://${description_pkg}/meshes/visual/link0.dae"/>
-        </geometry>
-      </visual>
-      <collision>
-        <geometry>
-          <mesh filename="package://${description_pkg}/meshes/collision/link0.stl"/>
-        </geometry>
-      </collision>
-      <inertial>
-        <origin xyz="${link0_cog}" rpy="0 0 0"/>
-        <mass value="${mass_link0}"/>
-        <inertia ixx="0.009" iyy="0.0122" izz="0.0122" ixy="0.0" ixz="-0.00010" iyz="0.0"/>
-      </inertial>
-    </link>
-    <link name="${arm_id}_link1">
-      <visual>
-        <geometry>
-          <mesh filename="package://${description_pkg}/meshes/visual/link1.dae"/>
-        </geometry>
-      </visual>
-      <collision>
-        <geometry>
-          <mesh filename="package://${description_pkg}/meshes/collision/link1.stl"/>
-        </geometry>
-      </collision>
-      <inertial>
-        <origin xyz="${link1_cog}" rpy="0 0 0"/>
-        <mass value="${mass_link1}"/>
-        <inertia ixx="0.01418" iyy="0.01181" izz="0.005515" ixy="0.0" ixz="0.0" iyz="0.00236"/>
-      </inertial>
-    </link>
-    <joint name="${arm_id}_joint1" type="revolute">
-      <safety_controller k_position="100.0" k_velocity="40.0" soft_lower_limit="-2.8973" soft_upper_limit="2.8973"/>
-      <origin rpy="0 0 0" xyz="0 0 0.333"/>
-      <parent link="${arm_id}_link0"/>
-      <child link="${arm_id}_link1"/>
-      <axis xyz="0 0 1"/>
-      <limit effort="87" lower="-2.8973" upper="2.8973" velocity="2.1750"/>
-      <dynamics damping="${joint_damping}"/>
-    </joint>
-    <link name="${arm_id}_link2">
-      <visual>
-        <geometry>
-          <mesh filename="package://${description_pkg}/meshes/visual/link2.dae"/>
-        </geometry>
-      </visual>
-      <collision>
-        <geometry>
-          <mesh filename="package://${description_pkg}/meshes/collision/link2.stl"/>
-        </geometry>
-      </collision>
-      <inertial>
-        <origin xyz="${link2_cog}" rpy="0 0 0"/>
-        <mass value="${mass_link2}"/>
-        <inertia ixx="0.014" ixy="0.0" ixz="0.0" iyy="0.0055" iyz="-0.0023" izz="0.01259"/>
-      </inertial>
-    </link>
-    <joint name="${arm_id}_joint2" type="revolute">
-      <safety_controller k_position="100.0" k_velocity="40.0" soft_lower_limit="-1.7628" soft_upper_limit="1.7628"/>
-      <origin rpy="${-pi/2} 0 0" xyz="0 0 0"/>
-      <parent link="${arm_id}_link1"/>
-      <child link="${arm_id}_link2"/>
-      <axis xyz="0 0 1"/>
-      <limit effort="87" lower="-1.7628" upper="1.7628" velocity="2.1750"/>
-      <dynamics damping="${joint_damping}"/>
-    </joint>
-    <link name="${arm_id}_link3">
-      <visual>
-        <geometry>
-          <mesh filename="package://${description_pkg}/meshes/visual/link3.dae"/>
-        </geometry>
-      </visual>
-      <collision>
-        <geometry>
-          <mesh filename="package://${description_pkg}/meshes/collision/link3.stl"/>
-        </geometry>
-      </collision>
-      <inertial>
-        <origin xyz="${link3_cog}" rpy="0 0 0"/>
-        <mass value="${mass_link3}"/>
-        <inertia ixx="0.00716" ixy="-0.00102" ixz="-0.02040" iyy="0.00920" iyz="-0.00102" izz="0.007159"/>
-      </inertial>
-    </link>
-    <joint name="${arm_id}_joint3" type="revolute">
-      <safety_controller k_position="100.0" k_velocity="40.0" soft_lower_limit="-2.8973" soft_upper_limit="2.8973"/>
-      <origin rpy="${pi/2} 0 0" xyz="0 -0.316 0"/>
-      <parent link="${arm_id}_link2"/>
-      <child link="${arm_id}_link3"/>
-      <axis xyz="0 0 1"/>
-      <limit effort="87" lower="-2.8973" upper="2.8973" velocity="2.1750"/>
-      <dynamics damping="${joint_damping}"/>
-    </joint>
-    <link name="${arm_id}_link4">
-      <visual>
-        <geometry>
-          <mesh filename="package://${description_pkg}/meshes/visual/link4.dae"/>
-        </geometry>
-      </visual>
-      <collision>
-        <geometry>
-          <mesh filename="package://${description_pkg}/meshes/collision/link4.stl"/>
-        </geometry>
-      </collision>
-      <inertial>
-        <origin xyz="${link4_cog}" rpy="0 0 0"/>
-        <mass value="${mass_link4}"/>
-        <inertia ixx="0.008164" ixy="0.003061" ixz="0.00102" iyy="0.008165" iyz="0.00102" izz="0.009185"/>
-      </inertial>
-    </link>
-    <joint name="${arm_id}_joint4" type="revolute">
-      <safety_controller k_position="100.0" k_velocity="40.0" soft_lower_limit="-3.0718" soft_upper_limit="-0.0698"/>
-      <origin rpy="${pi/2} 0 0" xyz="0.0825 0 0"/>
-      <parent link="${arm_id}_link3"/>
-      <child link="${arm_id}_link4"/>
-      <axis xyz="0 0 1"/>
-      <limit effort="87" lower="-3.0718" upper="-0.0698" velocity="2.1750"/>
-      <dynamics damping="${joint_damping}"/>
-    </joint>
-    <link name="${arm_id}_link5">
-      <visual>
-        <geometry>
-          <mesh filename="package://${description_pkg}/meshes/visual/link5.dae"/>
-        </geometry>
-      </visual>
-      <collision>
-        <geometry>
-          <mesh filename="package://${description_pkg}/meshes/collision/link5.stl"/>
-        </geometry>
-      </collision>
-      <inertial>
-        <origin xyz="${link5_cog}" rpy="0 0 0"/>
-        <mass value="${mass_link5}"/>
-        <inertia ixx="0.0307" ixy="0.0" ixz="0.0" iyy="0.02761" iyz="-0.0613" izz="0.00818"/>
-      </inertial>
-    </link>
-    <joint name="${arm_id}_joint5" type="revolute">
-      <safety_controller k_position="100.0" k_velocity="40.0" soft_lower_limit="-2.8973" soft_upper_limit="2.8973"/>
-      <origin rpy="${-pi/2} 0 0" xyz="-0.0825 0.384 0"/>
-      <parent link="${arm_id}_link4"/>
-      <child link="${arm_id}_link5"/>
-      <axis xyz="0 0 1"/>
-      <limit effort="12" lower="-2.8973" upper="2.8973" velocity="2.6100"/>
-      <dynamics damping="${joint_damping}"/>
-    </joint>
-    <link name="${arm_id}_link6">
-      <visual>
-        <geometry>
-          <mesh filename="package://${description_pkg}/meshes/visual/link6.dae"/>
-        </geometry>
-      </visual>
-      <collision>
-        <geometry>
-          <mesh filename="package://${description_pkg}/meshes/collision/link6.stl"/>
-        </geometry>
-      </collision>
-      <inertial>
-        <origin xyz="${link6_cog}" rpy="0 0 0"/>
-        <mass value="${mass_link6}"/>
-        <inertia ixx="0.00205" ixy="0.0" ixz="0.0" iyy="0.004089" iyz="0" izz="0.00490"/>
-      </inertial>
-    </link>
-    <joint name="${arm_id}_joint6" type="revolute">
-      <safety_controller k_position="100.0" k_velocity="40.0" soft_lower_limit="-0.0175" soft_upper_limit="3.7525"/>
-      <origin rpy="${pi/2} 0 0" xyz="0 0 0"/>
-      <parent link="${arm_id}_link5"/>
-      <child link="${arm_id}_link6"/>
-      <axis xyz="0 0 1"/>
-      <limit effort="12" lower="-0.0175" upper="3.7525" velocity="2.6100"/>
-      <dynamics damping="${joint_damping}"/>
-    </joint>
-    <link name="${arm_id}_link7">
-      <visual>
-        <geometry>
-          <mesh filename="package://${description_pkg}/meshes/visual/link7.dae"/>
-        </geometry>
-      </visual>
-      <collision>
-        <geometry>
-          <mesh filename="package://${description_pkg}/meshes/collision/link7.stl"/>
-        </geometry>
-      </collision>
-      <inertial>
-        <origin xyz="0 0 0" rpy="0 0 0"/>
-        <mass value="${mass_link7}"/>
-        <inertia ixx="0.3" ixy="0.0" ixz="0.0" iyy="0.3" iyz="0.0" izz="0.3"/>
-      </inertial>
-    </link>
-    <joint name="${arm_id}_joint7" type="revolute">
-      <safety_controller k_position="100.0" k_velocity="40.0" soft_lower_limit="-2.8973" soft_upper_limit="2.8973"/>
-      <origin rpy="${pi/2} 0 0" xyz="0.088 0 0"/>
-      <parent link="${arm_id}_link6"/>
-      <child link="${arm_id}_link7"/>
-      <axis xyz="0 0 1"/>
-      <limit effort="12" lower="-2.8973" upper="2.8973" velocity="2.6100"/>
-      <dynamics damping="${joint_damping}"/>
-    </joint>
-    <link name="${arm_id}_link8">
-      <inertial>
-        <origin xyz="0 0 0" rpy="0 0 0"/>
-        <mass value="${mass_link8}"/>
-        <inertia ixx="0.3" ixy="0.0" ixz="0.0" iyy="0.3" iyz="0.0" izz="0.3"/>
-      </inertial>
-    </link>
-    <joint name="${arm_id}_joint8" type="revolute">
-      <origin rpy="0 0 0" xyz="0 0 0.107"/>
-      <parent link="${arm_id}_link7"/>
-      <child link="${arm_id}_link8"/>
-      <axis xyz="0 0 1"/>
-      <limit effort="1" lower="0" upper="0.1" velocity="0.1"/>
-      <dynamics damping="100"/>
-    </joint>
+    </xacro:macro>
+    <xacro:macro name="panda_arm" params="arm_id:='panda' description_pkg:='franka_description' connected_to:='' xyz:='0 0 0' rpy:='0 0 0'">
+      <xacro:unless value="${not connected_to}">
+        <joint name="${arm_id}_joint_${connected_to}" type="fixed">
+          <parent link="${connected_to}"/>
+          <child link="${arm_id}_link0"/>
+          <origin rpy="${rpy}" xyz="${xyz}"/>
+        </joint>
+      </xacro:unless>
+      <xacro:property name="joint_damping" value="1.0"/>
+      <xacro:if value="${not connected_to}">
+        <joint name="robot_to_world" type="fixed">
+          <parent link="world" />
+          <child link="${arm_id}_link0" />
+          <origin xyz="0.0 0.0 0.0" rpy="0.0 0.0 0.0" />
+          <dynamics damping="${joint_damping}"/>
+        </joint>
+      </xacro:if>
+      <link name="${arm_id}_link0">
+        <visual>
+          <geometry>
+            <mesh filename="package://${description_pkg}/meshes/visual/link0.dae"/>
+          </geometry>
+        </visual>
+        <collision>
+          <geometry>
+            <mesh filename="package://${description_pkg}/meshes/collision/link0.stl"/>
+          </geometry>
+        </collision>
+        <inertial>
+          <origin xyz="${link0_cog}" rpy="0 0 0"/>
+          <mass value="${mass_link0}"/>
+          <inertia ixx="0.009" iyy="0.0122" izz="0.0122" ixy="0.0" ixz="-0.00010" iyz="0.0"/>
+        </inertial>
+      </link>
+      <link name="${arm_id}_link1">
+        <visual>
+          <geometry>
+            <mesh filename="package://${description_pkg}/meshes/visual/link1.dae"/>
+          </geometry>
+        </visual>
+        <collision>
+          <geometry>
+            <mesh filename="package://${description_pkg}/meshes/collision/link1.stl"/>
+          </geometry>
+        </collision>
+        <inertial>
+          <origin xyz="${link1_cog}" rpy="0 0 0"/>
+          <mass value="${mass_link1}"/>
+          <inertia ixx="0.01418" iyy="0.01181" izz="0.005515" ixy="0.0" ixz="0.0" iyz="0.00236"/>
+        </inertial>
+      </link>
+      <joint name="${arm_id}_joint1" type="revolute">
+        <safety_controller k_position="100.0" k_velocity="40.0" soft_lower_limit="-2.8973" soft_upper_limit="2.8973"/>
+        <origin rpy="0 0 0" xyz="0 0 0.333"/>
+        <parent link="${arm_id}_link0"/>
+        <child link="${arm_id}_link1"/>
+        <axis xyz="0 0 1"/>
+        <limit effort="87" lower="-2.8973" upper="2.8973" velocity="2.1750"/>
+        <dynamics damping="${joint_damping}"/>
+      </joint>
+      <link name="${arm_id}_link2">
+        <visual>
+          <geometry>
+            <mesh filename="package://${description_pkg}/meshes/visual/link2.dae"/>
+          </geometry>
+        </visual>
+        <collision>
+          <geometry>
+            <mesh filename="package://${description_pkg}/meshes/collision/link2.stl"/>
+          </geometry>
+        </collision>
+        <inertial>
+          <origin xyz="${link2_cog}" rpy="0 0 0"/>
+          <mass value="${mass_link2}"/>
+          <inertia ixx="0.014" ixy="0.0" ixz="0.0" iyy="0.0055" iyz="-0.0023" izz="0.01259"/>
+        </inertial>
+      </link>
+      <joint name="${arm_id}_joint2" type="revolute">
+        <safety_controller k_position="100.0" k_velocity="40.0" soft_lower_limit="-1.7628" soft_upper_limit="1.7628"/>
+        <origin rpy="${-pi/2} 0 0" xyz="0 0 0"/>
+        <parent link="${arm_id}_link1"/>
+        <child link="${arm_id}_link2"/>
+        <axis xyz="0 0 1"/>
+        <limit effort="87" lower="-1.7628" upper="1.7628" velocity="2.1750"/>
+        <dynamics damping="${joint_damping}"/>
+      </joint>
+      <link name="${arm_id}_link3">
+        <visual>
+          <geometry>
+            <mesh filename="package://${description_pkg}/meshes/visual/link3.dae"/>
+          </geometry>
+        </visual>
+        <collision>
+          <geometry>
+            <mesh filename="package://${description_pkg}/meshes/collision/link3.stl"/>
+          </geometry>
+        </collision>
+        <inertial>
+          <origin xyz="${link3_cog}" rpy="0 0 0"/>
+          <mass value="${mass_link3}"/>
+          <inertia ixx="0.00716" ixy="-0.00102" ixz="-0.02040" iyy="0.00920" iyz="-0.00102" izz="0.007159"/>
+        </inertial>
+      </link>
+      <joint name="${arm_id}_joint3" type="revolute">
+        <safety_controller k_position="100.0" k_velocity="40.0" soft_lower_limit="-2.8973" soft_upper_limit="2.8973"/>
+        <origin rpy="${pi/2} 0 0" xyz="0 -0.316 0"/>
+        <parent link="${arm_id}_link2"/>
+        <child link="${arm_id}_link3"/>
+        <axis xyz="0 0 1"/>
+        <limit effort="87" lower="-2.8973" upper="2.8973" velocity="2.1750"/>
+        <dynamics damping="${joint_damping}"/>
+      </joint>
+      <link name="${arm_id}_link4">
+        <visual>
+          <geometry>
+            <mesh filename="package://${description_pkg}/meshes/visual/link4.dae"/>
+          </geometry>
+        </visual>
+        <collision>
+          <geometry>
+            <mesh filename="package://${description_pkg}/meshes/collision/link4.stl"/>
+          </geometry>
+        </collision>
+        <inertial>
+          <origin xyz="${link4_cog}" rpy="0 0 0"/>
+          <mass value="${mass_link4}"/>
+          <inertia ixx="0.008164" ixy="0.003061" ixz="0.00102" iyy="0.008165" iyz="0.00102" izz="0.009185"/>
+        </inertial>
+      </link>
+      <joint name="${arm_id}_joint4" type="revolute">
+        <safety_controller k_position="100.0" k_velocity="40.0" soft_lower_limit="-3.0718" soft_upper_limit="-0.0698"/>
+        <origin rpy="${pi/2} 0 0" xyz="0.0825 0 0"/>
+        <parent link="${arm_id}_link3"/>
+        <child link="${arm_id}_link4"/>
+        <axis xyz="0 0 1"/>
+        <limit effort="87" lower="-3.0718" upper="-0.0698" velocity="2.1750"/>
+        <dynamics damping="${joint_damping}"/>
+      </joint>
+      <link name="${arm_id}_link5">
+        <visual>
+          <geometry>
+            <mesh filename="package://${description_pkg}/meshes/visual/link5.dae"/>
+          </geometry>
+        </visual>
+        <collision>
+          <geometry>
+            <mesh filename="package://${description_pkg}/meshes/collision/link5.stl"/>
+          </geometry>
+        </collision>
+        <inertial>
+          <origin xyz="${link5_cog}" rpy="0 0 0"/>
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